File: loop_single.kicad_sch (KiCad schematic)
At the start: 11 parts, among them J1 From Loop, J2 To Loop, SW1 Loopback, U1 6N139SDM, U2 GAQY211G2S

Commit message: rev a ready for go
Parts:
- D1: LCSC (none) -> C193012
- D2: LCSC (none) -> C7420372
- J1, J2: LCSC (none) -> C2997275
- R1: LCSC (none) -> C18724160
- R2, R3: LCSC (none) -> C4502
- R4: LCSC (none) -> C137262
- SW1: value Loopback -> THRU; LCSC (none) -> C54948
- U1: LCSC (none) -> C42186
- U2: LCSC (none) -> C7435104

Commit message: Rev b begin
Parts:
- removed D2: H5VL10B, local:SOD-882_L1.0-W0.6-BI, symbol local:H5VL10B
- added D2: SMF150CA_C519810, local:SMF_L2.9-W1.9-LS3.9-BI, symbol local:SMF150CA_C519810
- D1: value MB10FH5G0NP -> MB10S-50MIL; LCSC C193012 -> C2488; LCSC Part C193012 -> C2488
- J1, J2: footprint TerminalBlock_RND:TerminalBlock_RND_205-00045_1x02_P5.00mm_Horizontal -> local:TerminalBlock_5mm_labeled; LCSC Part (none) -> C2997275
- R1: value 150R 2W -> 47R 1W; footprint Resistor_SMD:R_1206_3216Metric -> Resistor_SMD:R_2512_6332Metric; LCSC C18724160 -> C341654; LCSC Part (none) -> C341654
- R2, R3: footprint Resistor_SMD:R_1206_3216Metric -> Resistor_SMD:R_0805_2012Metric; LCSC C4502 -> C17710; LCSC Part (none) -> C17710
- R4: footprint Resistor_SMD:R_1206_3216Metric -> Resistor_SMD:R_0805_2012Metric; LCSC C137262 -> C17673; LCSC Part (none) -> C17673
Connections:
- net at J2.1 (Pin_1), U2.4: now also D2.2
- net at J2.2 (Pin_2), SW1.1 (A1), U2.3: now also D2.1

Commit message: Thru-Hole version a go-go
Parts:
- D1: value MB10S-50MIL -> DF04MA; footprint local:MBF_L4.8-W3.9-P2.50-LS6.7-TR -> Diode_THT:Diode_Bridge_DIP-4_W7.62mm_P5.08mm; symbol local:MB10FH5G0NP -> Diode_Bridge:DF04M; LCSC C2488 -> (none); LCSC Part C2488 -> C193012; Mouser (none) -> 625-DF04MA-E3
- D2: value SMF150CA_C519810 -> 1.5KE180CAHE3_B/C; footprint local:SMF_L2.9-W1.9-LS3.9-BI -> Diode_THT:D_A-405_P10.16mm_Horizontal; symbol local:SMF150CA_C519810 -> PCM_Diode_TVS_AKL:D_TVS_Bidirectional_Generic
- R1: footprint Resistor_SMD:R_2512_6332Metric -> Resistor_THT:R_Axial_DIN0309_L9.0mm_D3.2mm_P12.70mm_Horizontal
- R2, R3, R4: footprint Resistor_SMD:R_0805_2012Metric -> Resistor_THT:R_Axial_DIN0204_L3.6mm_D1.6mm_P7.62mm_Horizontal
- SW1: footprint local:SW-SMD_DSIC01LSGET -> Button_Switch_THT:SW_DIP_SPSTx01_Slide_6.7x4.1mm_W7.62mm_P2.54mm_LowProfile; LCSC C54948 -> (none); LCSC Part C54948 -> (none); Mouser (none) -> 490-DS04-254-1S-01BK
- U1: value 6N139SDM -> 6N139M; footprint local:OPTO-SMD-8P_L9.6-W6.5-P2.54-LS10.0-BL -> Package_DIP:DIP-8_W10.16mm; LCSC C42186 -> (none); LCSC Part C42186 -> (none); Mouser (none) -> 512-6N139M
- U2: value GAQY211G2S -> AQY210EH; footprint local:SOP-4_L4.4-W4.0-P2.54-LS7.0-TL -> Package_DIP:DIP-4_W7.62mm; LCSC C7435104 -> (none); LCSC Part C7435104 -> (none); Mouser (none) -> 769-AQY210EH
Connections:
- net at J1.1 (Pin_1), R1.1, SW1.2 (A2): now also D1.4; no longer D1.2 (AC)
- net at U1.3 (VF-): now also D1.2 (-); no longer D1.3 (-)
- net at J1.2 (Pin_2), R1.2: now also D1.3; no longer D1.4 (AC)
Other:
- moved on the sheet: R2
