File: tty2040.kicad_sch (KiCad schematic)
At the start: 14 parts, among them U13 YC162-FR-072K4L, U14 YC162-FR-072K4L, U15 YC162-FR-072K4L

Commit message: rev a ready for go
Parts:
- LED1, LED2, LED3, LED4, LED5, LED6: LCSC (none) -> C2286
- U13, U14, U15: LCSC (none) -> C728827
Changed lines of the file:
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@@
+			)
+		)
+		(property "LCSC" "C2286"
+			(at 150.876 30.48 0)
+			(effects
+				(font
+					(size 1.27 1.27)
+				)
+				(hide yes)
 			)
 		)
@@
 			)
 		)
+		(property "LCSC" "C728827"
+			(at 163.83 48.26 0)
+			(effects
+				(font
+					(size 1.27 1.27)
+				)
+				(hide yes)
+			)
+		)
 		(pin "2"
 		)
@@
 			)
 		)
+		(property "LCSC" "C728827"
+			(at 163.83 34.29 0)
+			(effects
+				(font
+					(size 1.27 1.27)
+				)
+				(hide yes)
+			)
+		)
 		(pin "2"
 		)
@@
 			)
 		)
+		(property "LCSC" "C2286"
+			(at 150.876 22.86 0)
+			(effects
+				(font
+					(size 1.27 1.27)
+				)
+				(hide yes)
+			)
+		)
 		(pin "2"
 		)
@@
 			)
 		)
+		(property "LCSC" "C2286"
+			(at 150.876 58.42 0)
+			(effects
+				(font
+					(size 1.27 1.27)
+				)
+				(hide yes)
+			)
+		)
 		(pin "2"
 		)
@@
 		(property "LCSC Part" "C2286"
 			(at 147.32 52.07 0)
+			(effects
+				(font
+					(size 1.27 1.27)
+				)
+				(hide yes)
+			)
+		)
+		(property "LCSC" "C2286"
+			(at 150.876 36.83 0)
 			(effects
 				(font
@@
 			)
 		)
+		(property "LCSC" "C2286"
+			(at 150.876 50.8 0)
+			(effects
+				(font
+					(size 1.27 1.27)
+				)
+				(hide yes)
+			)
+		)
 		(pin "2"
 		)
@@
 		(property "LCSC Part" "C2286"
 			(at 147.32 59.69 0)
+			(effects
+				(font
+					(size 1.27 1.27)
+				)
+				(hide yes)
+			)
+		)
+		(property "LCSC" "C2286"
+			(at 150.876 44.45 0)
 			(effects
 				(font
@@
 			(effects
 				(font
+					(size 1.27 1.27)
+				)
+				(hide yes)
+			)
+		)
+		(property "LCSC" "C728827"
+			(at 163.83 20.32 0)
+			(effects
+				(font

Commit message: Initial gerbers (has issues)
Parts:
- added FID1, FID2: Fiducial, Fiducial:Fiducial_1mm_Mask3mm, symbol Mechanical:Fiducial
Changed lines of the file:
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@@
+	)
+	(symbol
+		(lib_id "Mechanical:Fiducial")
+		(at 36.83 21.59 0)
+		(unit 1)
+		(exclude_from_sim yes)
+		(in_bom no)
+		(on_board yes)
+		(dnp no)
+		(fields_autoplaced yes)
+		(property "Reference" "FID1"
+			(at 39.37 20.3199 0)
+			(effects
+				(font
+					(size 1.27 1.27)
+				)
+				(justify left)
+			)
+		)
+		(property "Value" "Fiducial"
+			(at 39.37 22.8599 0)
+			(effects
+				(font
+					(size 1.27 1.27)
+				)
+				(justify left)
+			)
+		)
+		(property "Footprint" "Fiducial:Fiducial_1mm_Mask3mm"
+			(at 36.83 21.59 0)
+			(effects
+				(font
+					(size 1.27 1.27)
+				)
+				(hide yes)
+			)
+		)
+		(property "Datasheet" "~"
+			(at 36.83 21.59 0)
+			(effects
+				(font
+					(size 1.27 1.27)
+				)
+				(hide yes)
+			)
+		)
+		(property "Description" "Fiducial Marker"
+			(at 36.83 21.59 0)
+			(effects
+				(font
+					(size 1.27 1.27)
+				)
+				(hide yes)
+			)
+		)
+		(instances
+			(project "tty2040"
+				(path "/abc27069-2ab3-4540-8984-2696f3591d8b"
+					(reference "FID1")
+					(unit 1)
+				)
+			)
+		)
 	)
 	(symbol
@@
 					(unit 1)
 				)
+			)
+		)
+	)
+	(symbol
+		(lib_id "Mechanical:Fiducial")
+		(at 36.83 16.51 0)
+		(unit 1)
+		(exclude_from_sim yes)
+		(in_bom no)
+		(on_board yes)
+		(dnp no)
+		(fields_autoplaced yes)
+		(property "Reference" "FID2"
+			(at 39.37 15.2399 0)
+			(effects
+				(font
+					(size 1.27 1.27)
+				)
+				(justify left)
+			)
+		)
+		(property "Value" "Fiducial"
+			(at 39.37 17.7799 0)
+			(effects
+				(font
+					(size 1.27 1.27)
+				)
+				(justify left)
+			)
+		)
+		(property "Footprint" "Fiducial:Fiducial_1mm_Mask3mm"
+			(at 36.83 16.51 0)
+			(effects
+				(font
+					(size 1.27 1.27)
+				)
+				(hide yes)
+			)
+		)
+		(property "Datasheet" "~"
+			(at 36.83 16.51 0)
+			(effects
+				(font
+					(size 1.27 1.27)
+				)
+				(hide yes)
+			)
+		)
+		(property "Description" "Fiducial Marker"
+			(at 36.83 16.51 0)
+			(effects
+				(font
+					(size 1.27 1.27)
+				)
+				(hide yes)
+			)
+		)
+		(instances
+			(project "tty2040"
+				(path "/abc27069-2ab3-4540-8984-2696f3591d8b"
+					(reference "FID2")
+					(unit 1)
+				)

Commit message: Rev b begin
Parts:
- removed U13, U14, U15: YC162-FR-072K4L, local:RES-ARRAY-SMD_0603-4P-L1.6-W1.6-BL, symbol local:YC162-FR-072K4L
- added R25, R26, R27, R28, R29, R30: 4.7K, Resistor_SMD:R_0805_2012Metric, symbol Device:R_Small
- LED1, LED2, LED3, LED4, LED5, LED6: footprint local:LED0603-RD -> Diode_SMD:D_0805_2012Metric; LCSC C2286 -> C2297; LCSC Part C2286 -> C2297
Connections:
- net ACT1: now also R25.2
- net ACT2: now also R26.2
- net ACT3: now also R27.2
- net ACT4: now also R28.2
- net ACT5: now also R29.2
- net ACT6: now also R30.2
- net at LED2.2 (A): now also R26.1
- net at LED5.2 (A): now also R29.1
- net at LED6.2 (A): now also R30.1
- net at LED3.2 (A): now also R27.1
- net at LED4.2 (A): now also R28.1
- net at LED1.2 (A): now also R25.1

Commit message: revB continue routing
Parts:
- A1: footprint Module_RaspberryPi_Pico:RaspberryPi_Pico_Common -> Module_RaspberryPi_Pico:RaspberryPi_Pico_Original_SMD_HandSolder
Changed lines of the file:
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@@
 			)
 		)
-		(property "Footprint" "Module_RaspberryPi_Pico:RaspberryPi_Pico_Common"
+		(property "Footprint" "Module_RaspberryPi_Pico:RaspberryPi_Pico_Original_SMD_HandSolder"
 			(at 99.06 149.86 0)
 			(effects

Commit message: Thru-Hole version a go-go
Parts:
- A1: footprint Module_RaspberryPi_Pico:RaspberryPi_Pico_Original_SMD_HandSolder -> Module_RaspberryPi_Pico:RaspberryPi_Pico_Common
- LED1: footprint Diode_SMD:D_0805_2012Metric -> LED_THT:LED_D3.0mm; symbol local:KT-0603R -> Device:LED; LCSC C2297 -> (none); LCSC Part C2297 -> (none)
- LED2, LED3, LED4, LED5, LED6: footprint Diode_SMD:D_0805_2012Metric -> LED_THT:LED_D3.0mm; symbol local:KT-0603R -> Device:LED
- R25, R26, R27, R28, R29, R30: footprint Resistor_SMD:R_0805_2012Metric -> Resistor_THT:R_Axial_DIN0204_L3.6mm_D1.6mm_P7.62mm_Horizontal
