File: tty2040.kicad_pcb (KiCad board)
At the start: 2 copper layers, 150.5 x 85.5 mm, 85 parts, among them J1 From Loop, J10 To Loop, J11 From Loop, J12 To Loop, J2 To Loop, J3 From Loop, J4 To Loop, J5 From Loop, J6 To Loop, J7 From Loop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

Commit message: revB continue routing
Parts:
- A1: footprint Module_RaspberryPi_Pico:RaspberryPi_Pico_Common -> Module_RaspberryPi_Pico:RaspberryPi_Pico_Original_SMD_HandSolder
- moved H3 143.0 mm to (205.8, 137.8)
- moved H4 138.4 mm to (205.6, 62.8)
- moved FID1 136.2 mm to (205.8, 131.8)
- moved H2 59.2 mm to (64.4, 138.2)
- moved FID2 36.8 mm to (69.8, 61.2)
- moved A1 19.0 mm to (82.5, 100.0), turned to 0 degrees
- moved H1 4.05 mm to (63.6, 61.2)
- moved D1 1.49 mm to (191.8, 79.8)
- moved D15 1.49 mm to (116.0, 75.7)
- moved D2 1.49 mm to (181.0, 75.8)
- moved D5 1.49 mm to (126.8, 79.7)
- moved J1 1.49 mm to (192.5, 68.0)
- moved J2 1.49 mm to (176.0, 68.0)
- moved J4 1.49 mm to (143.5, 68.0)
- moved J5 1.49 mm to (127.5, 68.0)
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Routing:
- net VCC: track 0.00 -> 145.2 mm
- net ACT6: track 0.00 -> 143.1 mm, vias 0 -> 2
- net /Loop1/FROM_LOOP: track 4.19 -> 137.9 mm, vias 0 -> 2
- net /Loop1/TO_LOOP: track 0.00 -> 126.5 mm, vias 0 -> 2
- net ACT1: track 0.00 -> 112.3 mm, vias 0 -> 2
- net ACT5: track 0.00 -> 107.1 mm, vias 0 -> 2
- net /Loop6/TO_LOOP: track 0.00 -> 104.3 mm, vias 0 -> 2
- net /Loop6/FROM_LOOP: track 4.19 -> 99.5 mm, vias 0 -> 2
- net ACT2: track 0.00 -> 88.7 mm, vias 0 -> 2
- net /Loop2/FROM_LOOP: track 4.19 -> 92.9 mm, vias 0 -> 2
- net ACT4: track 0.00 -> 87.1 mm, vias 0 -> 2
- net /Loop2/TO_LOOP: track 0.00 -> 82.7 mm, vias 0 -> 2
- net /Loop5/TO_LOOP: track 0.00 -> 76.2 mm
- net /Loop5/FROM_LOOP: track 4.19 -> 80.3 mm
- net /Loop4/FROM_LOOP: track 4.19 -> 64.3 mm, vias 0 -> 2
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Other:
- outline, holes or cut-outs redrawn

Commit message: Thru-Hole version a go-go
Parts:
- A1: footprint Module_RaspberryPi_Pico:RaspberryPi_Pico_Original_SMD_HandSolder -> Module_RaspberryPi_Pico:RaspberryPi_Pico_Common
- D1, D11, D3, D5, D7, D9: value MB10S-50MIL -> DF04MA; footprint local:MBF_L4.8-W3.9-P2.50-LS6.7-TR -> Diode_THT:Diode_Bridge_DIP-4_W7.62mm_P5.08mm
- D13, D15, D16, D17, D18, D2: value SMF150CA_C519810 -> 1.5KE180CAHE3_B/C; footprint local:SMF_L2.9-W1.9-LS3.9-BI -> Diode_THT:D_A-405_P10.16mm_Horizontal
- LED1, LED2, LED3, LED4, LED5, LED6: footprint Diode_SMD:D_0805_2012Metric -> LED_THT:LED_D3.0mm
- R1, R13, R17, R21, R5, R9: footprint Resistor_SMD:R_2512_6332Metric -> Resistor_THT:R_Axial_DIN0309_L9.0mm_D3.2mm_P12.70mm_Horizontal
- R10, R11, R12, R14, R15, R16, R18, R19, R2, R20, R22, R23, R24, R25, R26, R27, R28, R29, R3, R30, R4, R6, R7, R8: footprint Resistor_SMD:R_0805_2012Metric -> Resistor_THT:R_Axial_DIN0204_L3.6mm_D1.6mm_P7.62mm_Horizontal
- SW1, SW2, SW3, SW4, SW5, SW6: footprint local:SW-SMD_DSIC01LSGET -> Button_Switch_THT:SW_DIP_SPSTx01_Slide_6.7x4.1mm_W7.62mm_P2.54mm_LowProfile
- U1, U11, U3, U5, U7, U9: value 6N139SDM -> 6N139M; footprint local:OPTO-SMD-8P_L9.6-W6.5-P2.54-LS10.0-BL -> Package_DIP:DIP-8_W10.16mm
- U10, U12, U2, U4, U6, U8: value GAQY211G2S -> AQY210EH; footprint local:SOP-4_L4.4-W4.0-P2.54-LS7.0-TL -> Package_DIP:DIP-4_W7.62mm
- moved A1 95.7 mm to (178.0, 94.0), turned to -90 degrees
- moved FID1 93.9 mm to (210.0, 38.0)
- moved FID2 88.1 mm to (105.0, 142.0)
- moved R30 70.9 mm to (134.0, 94.8), turned to 90 degrees
- moved LED6 69.6 mm to (134.0, 100.3), turned to 90 degrees
- moved LED1 68.9 mm to (111.5, 100.3), turned to 90 degrees
- moved R25 66.4 mm to (111.5, 95.0), turned to 90 degrees
- moved H1 51.8 mm to (105.0, 30.0), turned to 0 degrees
- moved R29 46.5 mm to (129.5, 94.8), turned to 90 degrees
- moved LED5 44.4 mm to (129.5, 100.3), turned to 90 degrees
- moved H2 42.3 mm to (105.0, 150.0), turned to 0 degrees
- moved J1 38.2 mm to (195.9, 30.0)
- moved J3 38.1 mm to (162.9, 30.0)
- moved J2 38.1 mm to (178.5, 30.0)
- moved D2 38.1 mm to (186.0, 38.0)
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Connections:
- D1 pad 2: Net-(J1-Pin_1) -> Net-(D1--)
- D1 pad 3: Net-(D1--) -> Net-(J1-Pin_2)
- D1 pad 4: Net-(J1-Pin_2) -> Net-(J1-Pin_1)
- D11 pad 2: Net-(J11-Pin_1) -> Net-(D11--)
- D11 pad 3: Net-(D11--) -> Net-(J11-Pin_2)
- D11 pad 4: Net-(J11-Pin_2) -> Net-(J11-Pin_1)
- D3 pad 2: Net-(J3-Pin_1) -> Net-(D3--)
- D3 pad 3: Net-(D3--) -> Net-(J3-Pin_2)
- D3 pad 4: Net-(J3-Pin_2) -> Net-(J3-Pin_1)
- D5 pad 2: Net-(J5-Pin_1) -> Net-(D5--)
- D5 pad 3: Net-(D5--) -> Net-(J5-Pin_2)
- D5 pad 4: Net-(J5-Pin_2) -> Net-(J5-Pin_1)
- D7 pad 2: Net-(J7-Pin_1) -> Net-(D7--)
- D7 pad 3: Net-(D7--) -> Net-(J7-Pin_2)
- D7 pad 4: Net-(J7-Pin_2) -> Net-(J7-Pin_1)
- D9 pad 2: Net-(J9-Pin_1) -> Net-(D9--)
- D9 pad 3: Net-(D9--) -> Net-(J9-Pin_2)
- D9 pad 4: Net-(J9-Pin_2) -> Net-(J9-Pin_1)
Routing:
- net /Loop1/FROM_LOOP: track 137.9 -> 23.4 mm, vias 2 -> 0
- net ACT6: track 143.1 -> 38.3 mm, vias 2 -> 0
- net VCC: track 145.2 -> 245.8 mm
- net /Loop1/TO_LOOP: track 126.5 -> 44.5 mm, vias 2 -> 1
- net /Loop6/FROM_LOOP: track 99.5 -> 25.3 mm, vias 2 -> 0
- net ACT5: track 107.1 -> 46.2 mm, vias 2 -> 0
- net /Loop5/FROM_LOOP: track 80.3 -> 19.6 mm
- net /Loop6/TO_LOOP: track 104.3 -> 48.8 mm, vias 2 -> 0
- net /Loop2/FROM_LOOP: track 92.9 -> 38.9 mm, vias 2 -> 1
- net /Loop5/TO_LOOP: track 76.2 -> 29.3 mm
- net /Loop3/TO_LOOP: track 52.5 -> 85.8 mm, vias 2 -> 0
- net ACT4: track 87.1 -> 62.6 mm, vias 2 -> 1
- net /Loop2/TO_LOOP: track 82.7 -> 58.5 mm, vias 2 -> 0
- net /Loop4/TO_LOOP: track 56.7 -> 76.7 mm, vias 2 -> 0
- net ACT1: track 112.3 -> 98.8 mm, vias 2 -> 1
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- added copper zone on B.Cu, net GND
- removed copper zone on F.Cu, net GND
Other:
- board size 150.5 x 85.5 mm -> 115 x 135 mm
- board text added: "Connections Museum TTY Loop converter Revsion ${REVISION} Baked on ${CURRENT_DATE}"
- board text added: "Loop 3"
- board text added: "Loop 4"
- board text added: "Loop 5"
- board text added: "Loop 6"
- board text removed: "JLCJLCJLCJLC"
- board text removed: "Trans rights are human rights"

Commit message: rev B thru-hole prod
Routing:
- net VCC: track 245.8 -> 253.5 mm
Other:
- board size 115 x 135 mm -> 115 x 138 mm
- board text added: "JLCJLCJLCJLC"
- board text added: "Loop Activity"
Changed lines of the file:
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@@
 		(tags "Resistor Axial_DIN0204 series Axial Horizontal pin pitch 7.62mm 0.167W length 3.6mm diameter 1.6mm")
 		(property "Reference" "R4"
-			(at 3.81 -1.92 0)
+			(at 3.81 2 0)
 			(layer "F.SilkS")
 			(effects
@@
 		(tags "Resistor Axial_DIN0204 series Axial Horizontal pin pitch 7.62mm 0.167W length 3.6mm diameter 1.6mm")
 		(property "Reference" "R8"
-			(at 3.81 -1.92 0)
+			(at 9.42 0 0)
 			(layer "F.SilkS")
 			(effects
@@
 		(tags "Resistor Axial_DIN0204 series Axial Horizontal pin pitch 7.62mm 0.167W length 3.6mm diameter 1.6mm")
 		(property "Reference" "R12"
-			(at 3.81 -1.92 0)
+			(at 10.42 0 0)
 			(layer "F.SilkS")
 			(effects
@@
 	)
 	(gr_line
-		(start 105 22)
-		(end 210 22)
+		(start 105 21)
+		(end 210 21)
 		(stroke
 			(width 0.05)
@@
 	)
 	(gr_line
-		(start 100 152)
-		(end 100 27)
+		(start 100 154)
+		(end 100 26)
 		(stroke
 			(width 0.05)
@@
 	)
 	(gr_arc
-		(start 215 152)
-		(mid 213.535534 155.535534)
-		(end 210 157)
+		(start 215 154)
+		(mid 213.535534 157.535534)
+		(end 210 159)
 		(stroke
 			(width 0.05)
@@
 	)
 	(gr_line
-		(start 215 27)
+		(start 215 26)
 		(end 215 87)
 		(stroke
@@
 	(gr_line
 		(start 215 101)
-		(end 215 152)
+		(end 215 154)
 		(stroke
 			(width 0.05)
@@
 	)
 	(gr_arc
-		(start 105 157)
-		(mid 101.464466 155.535534)
-		(end 100 152)
+		(start 105 159)
+		(mid 101.464466 157.535534)
+		(end 100 154)
 		(stroke
 			(width 0.05)
@@
 	)
 	(gr_line
-		(start 210 157)
-		(end 105 157)
+		(start 210 159)
+		(end 105 159)
 		(stroke
 			(width 0.05)
@@
 	)
 	(gr_arc
-		(start 100 27)
-		(mid 101.464466 23.464466)
-		(end 105 22)
+		(start 100 26)
+		(mid 101.464466 22.464466)
+		(end 105 21)
 		(stroke
 			(width 0.05)
@@
 	)
 	(gr_arc
-		(start 210 22)
-		(mid 213.535534 23.464466)
-		(end 215 27)
+		(start 210 21)
+		(mid 213.535534 22.464466)
+		(end 215 26)
 		(stroke
 			(width 0.05)
@@
 		(layer "Edge.Cuts")
 	)
+	(gr_text "Loop Activity"
+		(at 116 105.5 0)
+		(layer "F.SilkS" knockout)
+		(effects
+			(font
+				(size 1.5 1.5)
+				(thickness 0.3)
+				(bold yes)
+			)
+			(justify left bottom)
+		)
+	)
 	(gr_text "Loop 1"
 		(at 188 41 -90)
@@
 		)
 	)
+	(gr_text "JLCJLCJLCJLC"
+		(at 162 90 0)
+		(layer "F.SilkS")
+		(effects
+			(font
+				(size 1.5 1.5)
+				(thickness 0.3)
+				(bold yes)
+			)
+			(justify left bottom)
+		)
+	)
 	(gr_text "Loop 4"
 		(at 123 123 270)
@@
 	)
 	(segment
-		(start 127.722943 64.71)
-		(end 112.8 79.632943)
+		(start 137.75 64)
+		(end 135.69 66.06)
 		(width 0.4)
 		(layer "B.Cu")
@@
 	)
 	(segment
-		(start 137.75 64)
-		(end 135.69 66.06)
+		(start 168.69 64.31)
+		(end 169 64)
 		(width 0.4)
 		(layer "B.Cu")
@@
 	)
 	(segment
-		(start 168.69 64.31)
-		(end 169 64)
+		(start 135.7 66.07)
+		(end 135.69 66.06)
 		(width 0.4)
 		(layer "B.Cu")
@@
 	)
 	(segment
-		(start 134.34 64.71)
-		(end 127.722943 64.71)
+		(start 169 64)
+		(end 137.75 64)
 		(width 0.4)
 		(layer "B.Cu")
@@
 	)
 	(segment
-		(start 135.7 66.07)
-		(end 135.69 66.06)
+		(start 112.8 68.2)
+		(end 112.8 109.74)
 		(width 0.4)
 		(layer "B.Cu")
@@
 	)
 	(segment
-		(start 169 64)
-		(end 137.75 64)
+		(start 112.8 109.74)
+		(end 111.54 111)
 		(width 0.4)
 		(layer "B.Cu")
@@
 	)
 	(segment
+		(start 133.13 63.5)
+		(end 117.5 63.5)
+		(width 0.4)
+		(layer "B.Cu")
+		(net 9)
+	)
+	(segment
 		(start 201.7 69)
 		(end 201.7 66.07)
@@
 	)
 	(segment
-		(start 135.69 66.06)
-		(end 134.34 64.71)
-		(width 0.4)
-		(layer "B.Cu")
-		(net 9)
-	)
-	(segment
 		(start 201.69 66.06)
 		(end 201.69 64.69)
@@
 	)
 	(segment
-		(start 112.8 79.632943)
-		(end 112.8 109.74)
+		(start 117.5 63.5)
+		(end 112.8 68.2)
 		(width 0.4)
 		(layer "B.Cu")
@@
 	)
 	(segment
-		(start 201.7 66.07)
-		(end 201.69 66.06)
+		(start 135.69 66.06)
+		(end 133.13 63.5)
 		(width 0.4)
 		(layer "B.Cu")
@@
 	)
 	(segment
-		(start 201 64)
-		(end 169 64)
+		(start 201.7 66.07)
+		(end 201.69 66.06)
 		(width 0.4)
 		(layer "B.Cu")
@@
 	)
 	(segment
-		(start 112.8 109.74)
-		(end 111.54 111)
+		(start 201 64)
+		(end 169 64)
 		(width 0.4)
 		(layer "B.Cu")
@@
 		(polygon
 			(pts
-				(xy 100 22) (xy 215 22) (xy 215 157) (xy 100 157)
+				(xy 100 21) (xy 215 21) (xy 215 159) (xy 100 159)
 			)
 		)
